File: BatterySystem/BatterySystem/BatterySystem.kicad_sch (KiCad schematic)
At the start: 0 parts

Commit message: Charger circuit gemaakt
Other:
- removed sheet BMS
Changed lines of the file:
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@@
 (kicad_sch (version 20230121) (generator eeschema)
   (paper "A4")
-  (sheet (at 114.3 86.36) (size 49.53 26.67) (fields_autoplaced)
+  (sheet (at 121.92 86.36) (size 49.53 26.67) (fields_autoplaced)
     (stroke (width 0.1524) (type solid))
     (fill (color 0 0 0 0.0000))
-    (property "Sheetname" "buckconv" (at 114.3 85.6484 0)
+    (property "Sheetname" "buckconv" (at 121.92 85.6484 0)
       (effects (font (size 1.27 1.27)) (justify left bottom))
     )
-    (property "Sheetfile" "buckconv.kicad_sch" (at 114.3 113.6146 0)
+    (property "Sheetfile" "buckconv.kicad_sch" (at 121.92 113.6146 0)
       (effects (font (size 1.27 1.27)) (justify left top))
     )
@@
     )
   )
-  (sheet (at 44.45 44.45) (size 44.45 26.67) (fields_autoplaced)
+  (sheet (at 201.93 85.09) (size 49.53 27.94) (fields_autoplaced)
     (stroke (width 0.1524) (type solid))
     (fill (color 0 0 0 0.0000))
-    (property "Sheetname" "BMS" (at 44.45 43.7384 0)
+    (property "Sheetname" "Charger" (at 201.93 84.3784 0)
       (effects (font (size 1.27 1.27)) (justify left bottom))
     )
-    (property "Sheetfile" "BMS.kicad_sch" (at 44.45 71.7046 0)
+    (property "Sheetfile" "charger.kicad_sch" (at 201.93 113.6146 0)
       (effects (font (size 1.27 1.27)) (justify left top))
     )
-    (instances
-      (project "BatterySystem"
-        (path "/087df5f5-f8bd-4aad-837d-9ee553cf1b81" (page "2"))
-      )
-    )
-  )
-  (sheet (at 114.3 44.45) (size 49.53 27.94) (fields_autoplaced)
-    (stroke (width 0.1524) (type solid))
-    (fill (color 0 0 0 0.0000))
-    (property "Sheetname" "Charger" (at 114.3 43.7384 0)
-      (effects (font (size 1.27 1.27)) (justify left bottom))
-    )
-    (property "Sheetfile" "charger.kicad_sch" (at 114.3 72.9746 0)
-      (effects (font (size 1.27 1.27)) (justify left top))
-    )
