File: BatterySystem/BatterySystem/usb.kicad_sch (KiCad schematic)
At the start: 0 parts

Commit message: Footprints toegevoegd aan battery charger
Parts:
- added U3: ~, VR20S3V3:USB-C 2.0 Female to DIP Adapter, symbol usbc:USBC-THT
Connections:
- new net D+: U3. (Vbus)
- new net D-: U3. (Vbus)
- new net GND: U3. (Vbus)
- new net Input: U3. (Vbus)
Changed lines of the file:
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@@
 (kicad_sch (version 20230121) (generator eeschema)
   (paper "A4")
+  (junction (at 104.14 87.63) (diameter 0) (color 0 0 0 0)
+  )
+  (wire (pts (xy 102.87 105.41) (xy 105.41 105.41))
+    (stroke (width 0) (type default))
+  )
+  (wire (pts (xy 102.87 99.06) (xy 105.41 99.06))
+    (stroke (width 0) (type default))
+  )
+  (wire (pts (xy 102.87 87.63) (xy 104.14 87.63))
+    (stroke (width 0) (type default))
+  )
+  (wire (pts (xy 102.87 93.98) (xy 105.41 93.98))
+    (stroke (width 0) (type default))
+  )
+  (wire (pts (xy 104.14 87.63) (xy 105.41 87.63))
+    (stroke (width 0) (type default))
+  )
+  (global_label "Input" (shape input) (at 105.41 105.41 0) (fields_autoplaced)
+    (effects (font (size 1.27 1.27)) (justify left))
+    (property "Intersheetrefs" "${INTERSHEET_REFS}" (at 113.0933 105.41 0)
+      (effects (font (size 1.27 1.27)) (justify left) hide)
+    )
+  )
+  (global_label "D+" (shape input) (at 105.41 93.98 0) (fields_autoplaced)
+    (effects (font (size 1.27 1.27)) (justify left))
+    (property "Intersheetrefs" "${INTERSHEET_REFS}" (at 111.1582 93.98 0)
+      (effects (font (size 1.27 1.27)) (justify left) hide)
+    )
+  )
+  (global_label "D-" (shape input) (at 105.41 99.06 0) (fields_autoplaced)
+    (effects (font (size 1.27 1.27)) (justify left))
+    (property "Intersheetrefs" "${INTERSHEET_REFS}" (at 111.1582 99.06 0)
+      (effects (font (size 1.27 1.27)) (justify left) hide)
+    )
+  )
+  (symbol (lib_id "usbc:USBC-THT") (at 91.44 91.44 0) (unit 1)
+    (in_bom yes) (on_board yes) (dnp no) (fields_autoplaced)
+    (property "Reference" "U3" (at 100.965 97.4718 0)
+      (effects (font (size 1.27 1.27)) (justify left))
+    )
+    (property "Value" "~" (at 91.44 91.44 0)
+      (effects (font (size 1.27 1.27)))
+    )
+    (property "Footprint" "VR20S3V3:USB-C 2.0 Female to DIP Adapter" (at 91.44 91.44 0)
+      (effects (font (size 1.27 1.27)) hide)
+    )
+    (property "Datasheet" "" (at 91.44 91.44 0)
+      (effects (font (size 1.27 1.27)) hide)
+    )
+    (pin "")
+    (pin "")
+    (pin "")
+    (pin "")
+    (instances
+      (project "BatterySystem"
+        (path "/087df5f5-f8bd-4aad-837d-9ee553cf1b81/c2cf6bc5-c7a7-4536-bd5f-b8479578647d"
+          (reference "U3") (unit 1)
+        )
+        (path "/087df5f5-f8bd-4aad-837d-9ee553cf1b81/f69338eb-3566-41cb-8f9e-7317d4388319"
+          (reference "U3") (unit 1)
+        )
+      )
+    )
+  )
+  (symbol (lib_id "power:PWR_FLAG") (at 104.14 87.63 0) (unit 1)
+    (in_bom yes) (on_board yes) (dnp no) (fields_autoplaced)
+    (property "Reference" "#FLG01" (at 104.14 85.725 0)
+      (effects (font (size 1.27 1.27)) hide)
+    )
+    (property "Value" "PWR_FLAG" (at 104.14 84.1281 0)
+      (effects (font (size 1.27 1.27)) hide)
+    )
+    (property "Footprint" "" (at 104.14 87.63 0)
+      (effects (font (size 1.27 1.27)) hide)
+    )
+    (property "Datasheet" "~" (at 104.14 87.63 0)
+      (effects (font (size 1.27 1.27)) hide)
+    )
+    (pin "1")
+    (instances
+      (project "BatterySystem"
+        (path "/087df5f5-f8bd-4aad-837d-9ee553cf1b81/c2cf6bc5-c7a7-4536-bd5f-b8479578647d"
+          (reference "#FLG01") (unit 1)
+        )
+        (path "/087df5f5-f8bd-4aad-837d-9ee553cf1b81/f69338eb-3566-41cb-8f9e-7317d4388319"
+          (reference "#FLG01") (unit 1)
+        )
+      )
+    )
+  )
+  (symbol (lib_id "power:GND") (at 105.41 87.63 0) (unit 1)
+    (in_bom yes) (on_board yes) (dnp no) (fields_autoplaced)
+    (property "Reference" "#PWR011" (at 105.41 93.98 0)
+      (effects (font (size 1.27 1.27)) hide)
+    )
+    (property "Value" "GND" (at 105.41 91.7655 0)
+      (effects (font (size 1.27 1.27)) hide)
+    )
+    (property "Footprint" "" (at 105.41 87.63 0)
+      (effects (font (size 1.27 1.27)) hide)
+    )
+    (property "Datasheet" "" (at 105.41 87.63 0)
+      (effects (font (size 1.27 1.27)) hide)
+    )
+    (pin "1")
+    (instances
+      (project "BatterySystem"
+        (path "/087df5f5-f8bd-4aad-837d-9ee553cf1b81/c2cf6bc5-c7a7-4536-bd5f-b8479578647d"
+          (reference "#PWR011") (unit 1)
+        )
+        (path "/087df5f5-f8bd-4aad-837d-9ee553cf1b81/f69338eb-3566-41cb-8f9e-7317d4388319"
+          (reference "#PWR011") (unit 1)
+        )
+      )
+    )
+  )
 )

Commit message: USB  connectie
Connections:
- net D+: now also U3.2 (D+); no longer U3. (Vbus)
- net D-: now also U3.3 (D-); no longer U3. (Vbus)
- net GND: now also U3.1 (GND); no longer U3. (Vbus)
- net Input: now also U3.4 (Vbus); no longer U3. (Vbus)
Changed lines of the file:
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@@
     (stroke (width 0) (type default))
   )
-  (global_label "Input" (shape input) (at 105.41 105.41 0) (fields_autoplaced)
+  (global_label "Input" (shape output) (at 105.41 105.41 0) (fields_autoplaced)
     (effects (font (size 1.27 1.27)) (justify left))
     (property "Intersheetrefs" "${INTERSHEET_REFS}" (at 113.0933 105.41 0)
@@
     )
   )
-  (global_label "D+" (shape input) (at 105.41 93.98 0) (fields_autoplaced)
+  (global_label "D+" (shape output) (at 105.41 93.98 0) (fields_autoplaced)
     (effects (font (size 1.27 1.27)) (justify left))
     (property "Intersheetrefs" "${INTERSHEET_REFS}" (at 111.1582 93.98 0)
@@
     )
   )
-  (global_label "D-" (shape input) (at 105.41 99.06 0) (fields_autoplaced)
+  (global_label "D-" (shape output) (at 105.41 99.06 0) (fields_autoplaced)
     (effects (font (size 1.27 1.27)) (justify left))
     (property "Intersheetrefs" "${INTERSHEET_REFS}" (at 111.1582 99.06 0)
@@
       (effects (font (size 1.27 1.27)) hide)
     )
-    (pin "")
-    (pin "")
-    (pin "")
-    (pin "")
+    (pin "2")
+    (pin "3")
+    (pin "1")
+    (pin "4")
     (instances
       (project "BatterySystem"
