File: BatterySystem/BatterySystem/buckconv.kicad_sch (KiCad schematic)
At the start: 10 parts, among them U1 3.3V

Commit message: Beetje gewerkt aan routen van de PCB en positioneren van componenten
Connections:
- net Vref: now reaches 3V3.1, C5.1, U1.3 (Vout)
Changed lines of the file:
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@@
   (junction (at 119.38 87.63) (diameter 0) (color 0 0 0 0)
+  )
+  (junction (at 161.29 87.63) (diameter 0) (color 0 0 0 0)
   )
   (junction (at 114.3 95.25) (diameter 0) (color 0 0 0 0)
@@
     (stroke (width 0) (type default))
   )
-  (wire (pts (xy 146.05 87.63) (xy 166.37 87.63))
+  (wire (pts (xy 146.05 87.63) (xy 161.29 87.63))
+    (stroke (width 0) (type default))
+  )
+  (wire (pts (xy 161.29 87.63) (xy 166.37 87.63))
     (stroke (width 0) (type default))
   )
   (wire (pts (xy 137.16 85.09) (xy 137.16 95.25))
+    (stroke (width 0) (type default))
+  )
+  (wire (pts (xy 161.29 86.995) (xy 161.29 87.63))
     (stroke (width 0) (type default))
   )
@@
     (stroke (width 0) (type default))
   )
+  (global_label "Vref" (shape input) (at 161.29 86.995 90) (fields_autoplaced)
+    (effects (font (size 1.27 1.27)) (justify left))
+    (property "Intersheetrefs" "${INTERSHEET_REFS}" (at 161.29 80.4001 90)
+      (effects (font (size 1.27 1.27)) (justify left) hide)
+    )
+  )
   (global_label "Bat" (shape input) (at 76.2 87.63 180) (fields_autoplaced)

Commit message: Buck converter gedaan en meer test point toegevoegd
Parts:
- F1: footprint (none) -> Fuse:Fuseholder_Clip-5x20mm_Eaton_1A5601-01_Inline_P20.80x6.76mm_D1.70mm_Horizontal
Changed lines of the file:
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@@
       (effects (font (size 1.27 1.27)))
     )
-    (property "Footprint" "" (at 87.63 89.408 90)
+    (property "Footprint" "Fuse:Fuseholder_Clip-5x20mm_Eaton_1A5601-01_Inline_P20.80x6.76mm_D1.70mm_Horizontal" (at 87.63 89.408 90)
       (effects (font (size 1.27 1.27)) hide)
     )
