File: Lichten-PCB/Connectoren.kicad_sch (KiCad schematic)
At the start: 0 parts

Commit message: Capacitor waardes toegevoegd en coonectoren toegevoegd
Parts:
- added J1: Conn_01x04_Socket, symbol Connector:Conn_01x04_Socket
Connections:
- new net 3V3: J1.1 (Pin_1)
- new net DIN: J1.3 (Pin_3)
- new net DOUT: J1.4 (Pin_4)
- new net GND: J1.2 (Pin_2)
Changed lines of the file:
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@@
 (kicad_sch (version 20230121) (generator eeschema)
   (paper "A4")
+  (junction (at 121.92 84.455) (diameter 0) (color 0 0 0 0)
+  )
+  (wire (pts (xy 118.745 84.455) (xy 121.92 84.455))
+    (stroke (width 0) (type default))
+  )
+  (wire (pts (xy 121.92 89.535) (xy 123.19 89.535))
+    (stroke (width 0) (type default))
+  )
+  (wire (pts (xy 121.92 84.455) (xy 123.19 84.455))
+    (stroke (width 0) (type default))
+  )
+  (wire (pts (xy 111.76 86.995) (xy 123.19 86.995))
+    (stroke (width 0) (type default))
+  )
+  (wire (pts (xy 116.84 92.075) (xy 123.19 92.075))
+    (stroke (width 0) (type default))
+  )
+  (rectangle (start 100.965 75.565) (end 154.94 100.33)
+    (stroke (width 0) (type default))
+    (fill (type none))
+  )
+  (text_box "De connector"
+    (at 100.965 100.33 0) (size 53.975 3.81)
+    (stroke (width 0) (type default))
+    (fill (type none))
+    (effects (font (size 1.27 1.27)) (justify left top))
+  )
+  (global_label "3V3" (shape input) (at 118.745 84.455 180) (fields_autoplaced)
+    (effects (font (size 1.27 1.27)) (justify right))
+    (property "Intersheetrefs" "${INTERSHEET_REFS}" (at 112.3316 84.455 0)
+      (effects (font (size 1.27 1.27)) (justify right) hide)
+    )
+  )
+  (global_label "DIN" (shape input) (at 121.92 89.535 180) (fields_autoplaced)
+    (effects (font (size 1.27 1.27)) (justify right))
+    (property "Intersheetrefs" "${INTERSHEET_REFS}" (at 115.8089 89.535 0)
+      (effects (font (size 1.27 1.27)) (justify right) hide)
+    )
+  )
+  (global_label "DOUT" (shape input) (at 116.84 92.075 180) (fields_autoplaced)
+    (effects (font (size 1.27 1.27)) (justify right))
+    (property "Intersheetrefs" "${INTERSHEET_REFS}" (at 109.0356 92.075 0)
+      (effects (font (size 1.27 1.27)) (justify right) hide)
+    )
+  )
+  (symbol (lib_id "power:GND") (at 111.76 86.995 0) (unit 1)
+    (in_bom yes) (on_board yes) (dnp no) (fields_autoplaced)
+    (property "Reference" "#PWR076" (at 111.76 93.345 0)
+      (effects (font (size 1.27 1.27)) hide)
+    )
+    (property "Value" "GND" (at 111.76 91.44 0)
+      (effects (font (size 1.27 1.27)) hide)
+    )
+    (property "Footprint" "" (at 111.76 86.995 0)
+      (effects (font (size 1.27 1.27)) hide)
+    )
+    (property "Datasheet" "" (at 111.76 86.995 0)
+      (effects (font (size 1.27 1.27)) hide)
+    )
+    (pin "1")
+    (instances
+      (project "Lichten-PCB"
+        (path "/1cd270d9-bf21-4eca-b51f-6d45fbba63ac/6a4346f3-a793-410a-9da0-631ae995a0da"
+          (reference "#PWR076") (unit 1)
+        )
+      )
+    )
+  )
+  (symbol (lib_id "power:PWR_FLAG") (at 121.92 84.455 0) (unit 1)
+    (in_bom yes) (on_board yes) (dnp no) (fields_autoplaced)
+    (property "Reference" "#FLG01" (at 121.92 82.55 0)
+      (effects (font (size 1.27 1.27)) hide)
+    )
+    (property "Value" "PWR_FLAG" (at 121.92 80.01 0)
+      (effects (font (size 1.27 1.27)))
+    )
+    (property "Footprint" "" (at 121.92 84.455 0)
+      (effects (font (size 1.27 1.27)) hide)
+    )
+    (property "Datasheet" "~" (at 121.92 84.455 0)
+      (effects (font (size 1.27 1.27)) hide)
+    )
+    (pin "1")
+    (instances
+      (project "Lichten-PCB"
+        (path "/1cd270d9-bf21-4eca-b51f-6d45fbba63ac/6a4346f3-a793-410a-9da0-631ae995a0da"
+          (reference "#FLG01") (unit 1)
+        )
+      )
+    )
+  )
+  (symbol (lib_id "Connector:Conn_01x04_Socket") (at 128.27 86.995 0) (unit 1)
+    (in_bom yes) (on_board yes) (dnp no) (fields_autoplaced)
+    (property "Reference" "J1" (at 129.54 86.995 0)
+      (effects (font (size 1.27 1.27)) (justify left))
+    )
+    (property "Value" "Conn_01x04_Socket" (at 129.54 89.535 0)
+      (effects (font (size 1.27 1.27)) (justify left))
+    )
+    (property "Footprint" "" (at 128.27 86.995 0)
+      (effects (font (size 1.27 1.27)) hide)
+    )
+    (property "Datasheet" "~" (at 128.27 86.995 0)
+      (effects (font (size 1.27 1.27)) hide)
+    )
+    (pin "1")
+    (pin "2")
+    (pin "3")
+    (pin "4")
+    (instances
+      (project "Lichten-PCB"
+        (path "/1cd270d9-bf21-4eca-b51f-6d45fbba63ac/6a4346f3-a793-410a-9da0-631ae995a0da"
+          (reference "J1") (unit 1)
+        )
+      )
+    )
+  )
 )

Commit message: Footprints toegevoegd
Parts:
- J1: footprint (none) -> Connector_PinHeader_2.54mm:PinHeader_1x04_P2.54mm_Vertical
Changed lines of the file:
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@@
       (effects (font (size 1.27 1.27)) (justify left))
     )
-    (property "Footprint" "" (at 128.27 86.995 0)
+    (property "Footprint" "Connector_PinHeader_2.54mm:PinHeader_1x04_P2.54mm_Vertical" (at 128.27 86.995 0)
       (effects (font (size 1.27 1.27)) hide)
     )

Commit message: Edge cuts en via toegevoegd met wat silk screen
Misschien op de achterkant een leuke foto van een aap
Connections:
- net DOUT: now also J1.2 (Pin_2); no longer J1.4 (Pin_4)
- net GND: now also J1.4 (Pin_4); no longer J1.2 (Pin_2)
- net 3V3 renamed +3V3
Changed lines of the file:
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@@
     (stroke (width 0) (type default))
   )
-  (wire (pts (xy 121.92 89.535) (xy 123.19 89.535))
+  (wire (pts (xy 118.745 89.535) (xy 123.19 89.535))
+    (stroke (width 0) (type default))
+  )
+  (wire (pts (xy 118.745 92.075) (xy 123.19 92.075))
     (stroke (width 0) (type default))
   )
@@
     (stroke (width 0) (type default))
   )
-  (wire (pts (xy 111.76 86.995) (xy 123.19 86.995))
-    (stroke (width 0) (type default))
-  )
-  (wire (pts (xy 116.84 92.075) (xy 123.19 92.075))
+  (wire (pts (xy 118.745 86.995) (xy 123.19 86.995))
     (stroke (width 0) (type default))
   )
@@
     (effects (font (size 1.27 1.27)) (justify left top))
   )
-  (global_label "3V3" (shape input) (at 118.745 84.455 180) (fields_autoplaced)
+  (global_label "+3V3" (shape input) (at 118.745 84.455 180) (fields_autoplaced)
     (effects (font (size 1.27 1.27)) (justify right))
-    (property "Intersheetrefs" "${INTERSHEET_REFS}" (at 112.3316 84.455 0)
+    (property "Intersheetrefs" "${INTERSHEET_REFS}" (at 110.7592 84.455 0)
       (effects (font (size 1.27 1.27)) (justify right) hide)
     )
   )
-  (global_label "DIN" (shape input) (at 121.92 89.535 180) (fields_autoplaced)
+  (global_label "DIN" (shape input) (at 118.745 89.535 180) (fields_autoplaced)
     (effects (font (size 1.27 1.27)) (justify right))
-    (property "Intersheetrefs" "${INTERSHEET_REFS}" (at 115.8089 89.535 0)
+    (property "Intersheetrefs" "${INTERSHEET_REFS}" (at 112.6339 89.535 0)
       (effects (font (size 1.27 1.27)) (justify right) hide)
     )
   )
-  (global_label "DOUT" (shape input) (at 116.84 92.075 180) (fields_autoplaced)
+  (global_label "DOUT" (shape input) (at 118.745 86.995 180) (fields_autoplaced)
     (effects (font (size 1.27 1.27)) (justify right))
-    (property "Intersheetrefs" "${INTERSHEET_REFS}" (at 109.0356 92.075 0)
+    (property "Intersheetrefs" "${INTERSHEET_REFS}" (at 110.9406 86.995 0)
       (effects (font (size 1.27 1.27)) (justify right) hide)
     )
   )
-  (symbol (lib_id "power:GND") (at 111.76 86.995 0) (unit 1)
+  (symbol (lib_id "power:GND") (at 118.745 92.075 0) (unit 1)
     (in_bom yes) (on_board yes) (dnp no) (fields_autoplaced)
-    (property "Reference" "#PWR076" (at 111.76 93.345 0)
+    (property "Reference" "#PWR076" (at 118.745 98.425 0)
       (effects (font (size 1.27 1.27)) hide)
     )
-    (property "Value" "GND" (at 111.76 91.44 0)
+    (property "Value" "GND" (at 118.745 96.52 0)
       (effects (font (size 1.27 1.27)) hide)
     )
-    (property "Footprint" "" (at 111.76 86.995 0)
+    (property "Footprint" "" (at 118.745 92.075 0)
       (effects (font (size 1.27 1.27)) hide)
     )
-    (property "Datasheet" "" (at 111.76 86.995 0)
+    (property "Datasheet" "" (at 118.745 92.075 0)
       (effects (font (size 1.27 1.27)) hide)
     )

Commit message: Trace dikte en mounting hole toegevoegd
Parts:
- added H1, H2, H3, H4: MountingHole_Pad, MountingHole:MountingHole_2.2mm_M2_DIN965_Pad, symbol Mechanical:MountingHole_Pad
Connections:
- net GND: now also H1.1, H2.1, H3.1, H4.1
Other:
- note added: "Mounting Hole"
Changed lines of the file:
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@@
 (kicad_sch (version 20230121) (generator eeschema)
-  (paper "A4")
+  (paper "A3")
+  (junction (at 121.92 92.075) (diameter 0) (color 0 0 0 0)
+  )
   (junction (at 121.92 84.455) (diameter 0) (color 0 0 0 0)
   )
@@
     (stroke (width 0) (type default))
   )
-  (wire (pts (xy 118.745 92.075) (xy 123.19 92.075))
+  (wire (pts (xy 121.92 92.075) (xy 123.19 92.075))
+    (stroke (width 0) (type default))
+  )
+  (wire (pts (xy 118.745 92.075) (xy 121.92 92.075))
     (stroke (width 0) (type default))
   )
@@
     (stroke (width 0) (type default))
   )
+  (rectangle (start 205.74 99.06) (end 245.11 102.87)
+    (stroke (width 0) (type default))
+    (fill (type none))
+  )
   (rectangle (start 100.965 75.565) (end 154.94 100.33)
+    (stroke (width 0) (type default))
+    (fill (type none))
+  )
+  (rectangle (start 205.74 73.66) (end 245.11 99.06)
     (stroke (width 0) (type default))
     (fill (type none))
@@
     (fill (type none))
     (effects (font (size 1.27 1.27)) (justify left top))
+  )
+  (text "Mounting Hole" (at 207.01 101.6 0)
+    (effects (font (size 1.27 1.27)) (justify left bottom))
   )
   (global_label "+3V3" (shape input) (at 118.745 84.455 180) (fields_autoplaced)
@@
     )
   )
+  (symbol (lib_id "power:GND") (at 210.82 81.28 0) (unit 1)
+    (in_bom yes) (on_board yes) (dnp no) (fields_autoplaced)
+    (property "Reference" "#PWR077" (at 210.82 87.63 0)
+      (effects (font (size 1.27 1.27)) hide)
+    )
+    (property "Value" "GND" (at 210.82 85.725 0)
+      (effects (font (size 1.27 1.27)) hide)
+    )
+    (property "Footprint" "" (at 210.82 81.28 0)
+      (effects (font (size 1.27 1.27)) hide)
+    )
+    (property "Datasheet" "" (at 210.82 81.28 0)
+      (effects (font (size 1.27 1.27)) hide)
+    )
+    (pin "1")
+    (instances
+      (project "Lichten-PCB"
+        (path "/1cd270d9-bf21-4eca-b51f-6d45fbba63ac/6a4346f3-a793-410a-9da0-631ae995a0da"
+          (reference "#PWR077") (unit 1)
+        )
+      )
+    )
+  )
+  (symbol (lib_id "power:PWR_FLAG") (at 121.92 92.075 180) (unit 1)
+    (in_bom yes) (on_board yes) (dnp no) (fields_autoplaced)
+    (property "Reference" "#FLG02" (at 121.92 93.98 0)
+      (effects (font (size 1.27 1.27)) hide)
+    )
+    (property "Value" "PWR_FLAG" (at 121.92 96.2105 0)
+      (effects (font (size 1.27 1.27)) hide)
+    )
+    (property "Footprint" "" (at 121.92 92.075 0)
+      (effects (font (size 1.27 1.27)) hide)
+    )
+    (property "Datasheet" "~" (at 121.92 92.075 0)
+      (effects (font (size 1.27 1.27)) hide)
+    )
+    (pin "1")
+    (instances
+      (project "Lichten-PCB"
+        (path "/1cd270d9-bf21-4eca-b51f-6d45fbba63ac/6a4346f3-a793-410a-9da0-631ae995a0da"
+          (reference "#FLG02") (unit 1)
+        )
+      )
+    )
+  )
   (symbol (lib_id "power:GND") (at 118.745 92.075 0) (unit 1)
     (in_bom yes) (on_board yes) (dnp no) (fields_autoplaced)
@@
     )
     (property "Value" "PWR_FLAG" (at 121.92 80.01 0)
-      (effects (font (size 1.27 1.27)))
+      (effects (font (size 1.27 1.27)) hide)
     )
     (property "Footprint" "" (at 121.92 84.455 0)
@@
     )
   )
+  (symbol (lib_id "power:GND") (at 234.95 81.28 0) (unit 1)
+    (in_bom yes) (on_board yes) (dnp no) (fields_autoplaced)
+    (property "Reference" "#PWR079" (at 234.95 87.63 0)
+      (effects (font (size 1.27 1.27)) hide)
+    )
+    (property "Value" "GND" (at 234.95 85.725 0)
+      (effects (font (size 1.27 1.27)) hide)
+    )
+    (property "Footprint" "" (at 234.95 81.28 0)
+      (effects (font (size 1.27 1.27)) hide)
+    )
+    (property "Datasheet" "" (at 234.95 81.28 0)
+      (effects (font (size 1.27 1.27)) hide)
+    )
+    (pin "1")
+    (instances
+      (project "Lichten-PCB"
+        (path "/1cd270d9-bf21-4eca-b51f-6d45fbba63ac/6a4346f3-a793-410a-9da0-631ae995a0da"
+          (reference "#PWR079") (unit 1)
+        )
+      )
+    )
+  )
+  (symbol (lib_id "power:GND") (at 234.95 93.98 0) (unit 1)
+    (in_bom yes) (on_board yes) (dnp no) (fields_autoplaced)
+    (property "Reference" "#PWR080" (at 234.95 100.33 0)
+      (effects (font (size 1.27 1.27)) hide)
+    )
+    (property "Value" "GND" (at 234.95 98.425 0)
+      (effects (font (size 1.27 1.27)) hide)
+    )
+    (property "Footprint" "" (at 234.95 93.98 0)
+      (effects (font (size 1.27 1.27)) hide)
+    )
+    (property "Datasheet" "" (at 234.95 93.98 0)
+      (effects (font (size 1.27 1.27)) hide)
+    )
+    (pin "1")
+    (instances
+      (project "Lichten-PCB"
+        (path "/1cd270d9-bf21-4eca-b51f-6d45fbba63ac/6a4346f3-a793-410a-9da0-631ae995a0da"
+          (reference "#PWR080") (unit 1)
+        )
+      )
+    )
+  )
   (symbol (lib_id "Connector:Conn_01x04_Socket") (at 128.27 86.995 0) (unit 1)
     (in_bom yes) (on_board yes) (dnp no) (fields_autoplaced)
-    (property "Reference" "J1" (at 129.54 86.995 0)
+    (property "Reference" "J1" (at 128.9812 88.5818 0)
       (effects (font (size 1.27 1.27)) (justify left))
     )
     (property "Value" "Conn_01x04_Socket" (at 129.54 89.535 0)
-      (effects (font (size 1.27 1.27)) (justify left))
+      (effects (font (size 1.27 1.27)) (justify left) hide)
     )
     (property "Footprint" "Connector_PinHeader_2.54mm:PinHeader_1x04_P2.54mm_Vertical" (at 128.27 86.995 0)
@@
         )
       )
+    )
+  )
+  (symbol (lib_id "Mechanical:MountingHole_Pad") (at 210.82 91.44 0) (unit 1)
+    (in_bom yes) (on_board yes) (dnp no) (fields_autoplaced)
+    (property "Reference" "H2" (at 213.36 90.4868 0)
+      (effects (font (size 1.27 1.27)) (justify left))
+    )
+    (property "Value" "MountingHole_Pad" (at 213.36 91.4473 0)
+      (effects (font (size 1.27 1.27)) (justify left) hide)
+    )
+    (property "Footprint" "MountingHole:MountingHole_2.2mm_M2_DIN965_Pad" (at 210.82 91.44 0)
+      (effects (font (size 1.27 1.27)) hide)
+    )
+    (property "Datasheet" "~" (at 210.82 91.44 0)
+      (effects (font (size 1.27 1.27)) hide)
+    )
+    (pin "1")
+    (instances
+      (project "Lichten-PCB"
+        (path "/1cd270d9-bf21-4eca-b51f-6d45fbba63ac/6a4346f3-a793-410a-9da0-631ae995a0da"
+          (reference "H2") (unit 1)
+        )
+      )
+    )
+  )
+  (symbol (lib_id "Mechanical:MountingHole_Pad") (at 234.95 91.44 0) (unit 1)
+    (in_bom yes) (on_board yes) (dnp no) (fields_autoplaced)
+    (property "Reference" "H4" (at 237.49 90.4868 0)
+      (effects (font (size 1.27 1.27)) (justify left))
+    )
+    (property "Value" "MountingHole_Pad" (at 237.49 91.4473 0)
+      (effects (font (size 1.27 1.27)) (justify left) hide)
+    )
+    (property "Footprint" "MountingHole:MountingHole_2.2mm_M2_DIN965_Pad" (at 234.95 91.44 0)
+      (effects (font (size 1.27 1.27)) hide)
+    )
+    (property "Datasheet" "~" (at 234.95 91.44 0)
+      (effects (font (size 1.27 1.27)) hide)
+    )
+    (pin "1")
+    (instances
+      (project "Lichten-PCB"
+        (path "/1cd270d9-bf21-4eca-b51f-6d45fbba63ac/6a4346f3-a793-410a-9da0-631ae995a0da"
+          (reference "H4") (unit 1)
+        )
+      )
+    )
+  )
+  (symbol (lib_id "Mechanical:MountingHole_Pad") (at 210.82 78.74 0) (unit 1)
+    (in_bom yes) (on_board yes) (dnp no) (fields_autoplaced)
+    (property "Reference" "H1" (at 213.36 77.7868 0)
+      (effects (font (size 1.27 1.27)) (justify left))
+    )
+    (property "Value" "MountingHole_Pad" (at 213.36 78.7473 0)
+      (effects (font (size 1.27 1.27)) (justify left) hide)
+    )
+    (property "Footprint" "MountingHole:MountingHole_2.2mm_M2_DIN965_Pad" (at 210.82 78.74 0)
+      (effects (font (size 1.27 1.27)) hide)
+    )
+    (property "Datasheet" "~" (at 210.82 78.74 0)
+      (effects (font (size 1.27 1.27)) hide)
+    )
+    (pin "1")
+    (instances
+      (project "Lichten-PCB"
+        (path "/1cd270d9-bf21-4eca-b51f-6d45fbba63ac/6a4346f3-a793-410a-9da0-631ae995a0da"
+          (reference "H1") (unit 1)
+        )
+      )
+    )
+  )
+  (symbol (lib_id "Mechanical:MountingHole_Pad") (at 234.95 78.74 0) (unit 1)
+    (in_bom yes) (on_board yes) (dnp no) (fields_autoplaced)
+    (property "Reference" "H3" (at 237.49 77.7868 0)
+      (effects (font (size 1.27 1.27)) (justify left))
+    )
+    (property "Value" "MountingHole_Pad" (at 237.49 78.7473 0)
+      (effects (font (size 1.27 1.27)) (justify left) hide)
+    )
+    (property "Footprint" "MountingHole:MountingHole_2.2mm_M2_DIN965_Pad" (at 234.95 78.74 0)
+      (effects (font (size 1.27 1.27)) hide)
+    )
+    (property "Datasheet" "~" (at 234.95 78.74 0)
+      (effects (font (size 1.27 1.27)) hide)
+    )
+    (pin "1")
+    (instances
+      (project "Lichten-PCB"
+        (path "/1cd270d9-bf21-4eca-b51f-6d45fbba63ac/6a4346f3-a793-410a-9da0-631ae995a0da"
+          (reference "H3") (unit 1)
+        )
+      )
+    )
+  )
+  (symbol (lib_id "power:GND") (at 210.82 93.98 0) (unit 1)
+    (in_bom yes) (on_board yes) (dnp no) (fields_autoplaced)
+    (property "Reference" "#PWR078" (at 210.82 100.33 0)
+      (effects (font (size 1.27 1.27)) hide)
+    )
+    (property "Value" "GND" (at 210.82 98.425 0)
+      (effects (font (size 1.27 1.27)) hide)
+    )
+    (property "Footprint" "" (at 210.82 93.98 0)
+      (effects (font (size 1.27 1.27)) hide)
+    )
+    (property "Datasheet" "" (at 210.82 93.98 0)
+      (effects (font (size 1.27 1.27)) hide)
+    )
+    (pin "1")
+    (instances
+      (project "Lichten-PCB"
+        (path "/1cd270d9-bf21-4eca-b51f-6d45fbba63ac/6a4346f3-a793-410a-9da0-631ae995a0da"
+          (reference "#PWR078") (unit 1)
+        )
+      )

Commit message: 3D van connector toegevoegd
Parts:
- J1: footprint Connector_PinHeader_2.54mm:PinHeader_1x04_P2.54mm_Vertical -> TerminalBlock_4Ucon:TerminalBlock_4Ucon_1x04_P3.50mm_Horizontal
Changed lines of the file:
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@@
       (effects (font (size 1.27 1.27)) (justify left) hide)
     )
-    (property "Footprint" "Connector_PinHeader_2.54mm:PinHeader_1x04_P2.54mm_Vertical" (at 128.27 86.995 0)
+    (property "Footprint" "TerminalBlock_4Ucon:TerminalBlock_4Ucon_1x04_P3.50mm_Horizontal" (at 128.27 86.995 0)
       (effects (font (size 1.27 1.27)) hide)
     )
