File: PCB-light-challenge/PIR.kicad_sch (KiCad schematic)
At the start: 0 parts

Commit message: Merge branch 'main' of https://github.com/ayoub070/Light-challenge
Parts:
- added PIR_sens1: ~, PIRsens:PIR-SENS, symbol PIRsens:PIR
Connections:
- new net +3V3: PIR_sens1.1 (VCC)
- new net GND: PIR_sens1.2 (GND)
- new net OUT DATA: PIR_sens1.3 (OUT_data)
Changed lines of the file:
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@@
 (kicad_sch (version 20230121) (generator eeschema)
   (paper "A4")
+  (wire (pts (xy 135.89 80.01) (xy 135.89 87.63))
+    (stroke (width 0) (type default))
+  )
+  (wire (pts (xy 114.935 81.915) (xy 114.935 82.55))
+    (stroke (width 0) (type default))
+  )
+  (wire (pts (xy 130.81 80.01) (xy 130.81 82.55))
+    (stroke (width 0) (type default))
+  )
+  (wire (pts (xy 140.97 80.01) (xy 140.97 92.71))
+    (stroke (width 0) (type default))
+  )
+  (wire (pts (xy 114.935 92.71) (xy 140.97 92.71))
+    (stroke (width 0) (type default))
+  )
+  (wire (pts (xy 114.935 87.63) (xy 135.89 87.63))
+    (stroke (width 0) (type default))
+  )
+  (wire (pts (xy 114.935 82.55) (xy 130.81 82.55))
+    (stroke (width 0) (type default))
+  )
+  (global_label "OUT DATA" (shape output) (at 114.935 92.71 180) (fields_autoplaced)
+    (effects (font (size 1.27 1.27)) (justify right))
+    (property "Intersheetrefs" "${INTERSHEET_REFS}" (at 103.2238 92.71 0)
+      (effects (font (size 1.27 1.27)) (justify right) hide)
+    )
+  )
+  (symbol (lib_id "power:+3V3") (at 114.935 81.915 0) (unit 1)
+    (in_bom yes) (on_board yes) (dnp no) (fields_autoplaced)
+    (property "Reference" "#PWR016" (at 114.935 85.725 0)
+      (effects (font (size 1.27 1.27)) hide)
+    )
+    (property "Value" "+3V3" (at 114.935 78.4131 0)
+      (effects (font (size 1.27 1.27)))
+    )
+    (property "Footprint" "" (at 114.935 81.915 0)
+      (effects (font (size 1.27 1.27)) hide)
+    )
+    (property "Datasheet" "" (at 114.935 81.915 0)
+      (effects (font (size 1.27 1.27)) hide)
+    )
+    (pin "1")
+    (instances
+      (project "PCB-light-challenge"
+        (path "/35573e8f-7834-430c-81d2-239f316c7834/5679ea21-1e58-482d-afee-07308fc996bf"
+          (reference "#PWR016") (unit 1)
+        )
+      )
+    )
+  )
+  (symbol (lib_id "PIRsens:PIR") (at 135.89 68.58 0) (unit 1)
+    (in_bom yes) (on_board yes) (dnp no)
+    (property "Reference" "PIR_sens1" (at 132.715 64.135 0)
+      (effects (font (size 1.27 1.27)) (justify left))
+    )
+    (property "Value" "~" (at 135.89 68.58 0)
+      (effects (font (size 1.27 1.27)))
+    )
+    (property "Footprint" "PIRsens:PIR-SENS" (at 135.89 68.58 0)
+      (effects (font (size 1.27 1.27)) hide)
+    )
+    (property "Datasheet" "" (at 135.89 68.58 0)
+      (effects (font (size 1.27 1.27)) hide)
+    )
+    (pin "1")
+    (pin "2")
+    (pin "3")
+    (instances
+      (project "PCB-light-challenge"
+        (path "/35573e8f-7834-430c-81d2-239f316c7834/5679ea21-1e58-482d-afee-07308fc996bf"
+          (reference "PIR_sens1") (unit 1)
+        )
+      )
+    )
+  )
+  (symbol (lib_id "power:GND") (at 114.935 87.63 0) (unit 1)
+    (in_bom yes) (on_board yes) (dnp no) (fields_autoplaced)
+    (property "Reference" "#PWR017" (at 114.935 93.98 0)
+      (effects (font (size 1.27 1.27)) hide)
+    )
+    (property "Value" "GND" (at 114.935 91.7655 0)
+      (effects (font (size 1.27 1.27)) hide)
+    )
+    (property "Footprint" "" (at 114.935 87.63 0)
+      (effects (font (size 1.27 1.27)) hide)
+    )
+    (property "Datasheet" "" (at 114.935 87.63 0)
+      (effects (font (size 1.27 1.27)) hide)
+    )
+    (pin "1")
+    (instances
+      (project "PCB-light-challenge"
+        (path "/35573e8f-7834-430c-81d2-239f316c7834/5679ea21-1e58-482d-afee-07308fc996bf"
+          (reference "#PWR017") (unit 1)
+        )
+      )
+    )
+  )
 )
