File: PCB-light-challenge/PIR.kicad_sch (KiCad schematic)
At the start: 2 parts

Commit message: TP footprint verandert,  apparte grond (P-) gemaakt.  AC  clearance verandert.  connector voor PIR verandert
Connections:
- net GND renamed P-
Changed lines of the file:
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@@
+    )
+  )
+  (global_label "P-" (shape input) (at 135.128 64.262 180) (fields_autoplaced)
+    (effects (font (size 1.27 1.27)) (justify right))
+    (property "Intersheetrefs" "${INTERSHEET_REFS}" (at 129.3798 64.262 0)
+      (effects (font (size 1.27 1.27)) (justify right) hide)
     )
   )
@@
     (effects (font (size 1.27 1.27)) (justify right))
     (property "Intersheetrefs" "${INTERSHEET_REFS}" (at 128.7146 59.182 0)
+      (effects (font (size 1.27 1.27)) (justify right) hide)
+    )
+  )
+  (global_label "P-" (shape input) (at 81.915 64.77 180) (fields_autoplaced)
+    (effects (font (size 1.27 1.27)) (justify right))
+    (property "Intersheetrefs" "${INTERSHEET_REFS}" (at 76.1668 64.77 0)
       (effects (font (size 1.27 1.27)) (justify right) hide)
     )
@@
         )
       )
-    )
-  )
-  (symbol (lib_id "power:GND") (at 135.128 64.262 0) (unit 1)
-    (in_bom yes) (on_board yes) (dnp no) (fields_autoplaced)
-    (property "Reference" "#PWR03" (at 135.128 70.612 0)
-      (effects (font (size 1.27 1.27)) hide)
-    )
-    (property "Value" "GND" (at 135.128 68.3975 0)
-      (effects (font (size 1.27 1.27)) hide)
-    )
-    (property "Footprint" "" (at 135.128 64.262 0)
-      (effects (font (size 1.27 1.27)) hide)
-    )
-    (property "Datasheet" "" (at 135.128 64.262 0)
-      (effects (font (size 1.27 1.27)) hide)
-    )
-    (pin "1")
-    (instances
-      (project "PCB-light-challenge"
-        (path "/35573e8f-7834-430c-81d2-239f316c7834/5679ea21-1e58-482d-afee-07308fc996bf"
-          (reference "#PWR03") (unit 1)
-        )
-      )
-    )
-  )
-  (symbol (lib_id "power:GND") (at 81.915 64.77 0) (unit 1)
-    (in_bom yes) (on_board yes) (dnp no) (fields_autoplaced)
-    (property "Reference" "#PWR017" (at 81.915 71.12 0)
-      (effects (font (size 1.27 1.27)) hide)
-    )
-    (property "Value" "GND" (at 81.915 68.9055 0)
-      (effects (font (size 1.27 1.27)) hide)
-    )
-    (property "Footprint" "" (at 81.915 64.77 0)
-      (effects (font (size 1.27 1.27)) hide)
-    )
-    (property "Datasheet" "" (at 81.915 64.77 0)
-      (effects (font (size 1.27 1.27)) hide)
-    )
-    (pin "1")
-    (instances
-      (project "PCB-light-challenge"
-        (path "/35573e8f-7834-430c-81d2-239f316c7834/5679ea21-1e58-482d-afee-07308fc996bf"
-          (reference "#PWR017") (unit 1)
-        )
-      )

Commit message: Vias  kleiner gemaakt en grond GND genoemd op silkscreen
Parts:
- renumbered PIR_sens1 to PIR1, PIR_sens2 to PIR2
Connections:
- net GP1 renamed GP19
- net GP2 renamed GP20
Changed lines of the file:
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@@
     (stroke (width 0) (type default))
   )
-  (global_label "GP1" (shape output) (at 81.915 69.85 180) (fields_autoplaced)
+  (global_label "GP19" (shape output) (at 81.915 69.85 180) (fields_autoplaced)
     (effects (font (size 1.27 1.27)) (justify right))
-    (property "Intersheetrefs" "${INTERSHEET_REFS}" (at 75.2597 69.85 0)
+    (property "Intersheetrefs" "${INTERSHEET_REFS}" (at 74.0502 69.85 0)
       (effects (font (size 1.27 1.27)) (justify right) hide)
     )
@@
     )
   )
-  (global_label "GP2" (shape output) (at 135.128 69.342 180) (fields_autoplaced)
+  (global_label "GP20" (shape output) (at 135.128 69.342 180) (fields_autoplaced)
     (effects (font (size 1.27 1.27)) (justify right))
-    (property "Intersheetrefs" "${INTERSHEET_REFS}" (at 128.4727 69.342 0)
+    (property "Intersheetrefs" "${INTERSHEET_REFS}" (at 127.2632 69.342 0)
       (effects (font (size 1.27 1.27)) (justify right) hide)
     )
@@
   (symbol (lib_id "PIRsens:PIR") (at 156.083 45.212 0) (unit 1)
     (in_bom yes) (on_board yes) (dnp no)
-    (property "Reference" "PIR_sens2" (at 152.908 40.767 0)
+    (property "Reference" "PIR2" (at 152.908 40.767 0)
       (effects (font (size 1.27 1.27)) (justify left))
     )
@@
       (project "PCB-light-challenge"
         (path "/35573e8f-7834-430c-81d2-239f316c7834/5679ea21-1e58-482d-afee-07308fc996bf"
-          (reference "PIR_sens2") (unit 1)
+          (reference "PIR2") (unit 1)
         )
       )
     )
   )
-  (symbol (lib_id "PIRsens:PIR") (at 102.87 45.72 0) (unit 1)
+  (symbol (lib_name "PIR_1") (lib_id "PIRsens:PIR") (at 102.87 45.72 0) (unit 1)
     (in_bom yes) (on_board yes) (dnp no)
-    (property "Reference" "PIR_sens1" (at 99.695 41.275 0)
+    (property "Reference" "PIR1" (at 99.695 41.275 0)
       (effects (font (size 1.27 1.27)) (justify left))
     )
@@
       (project "PCB-light-challenge"
         (path "/35573e8f-7834-430c-81d2-239f316c7834/5679ea21-1e58-482d-afee-07308fc996bf"
-          (reference "PIR_sens1") (unit 1)
+          (reference "PIR1") (unit 1)
         )
       )

Commit message: 3V3 OUT voor RGB toegevoegd en footprint van connectoren verandert naar JST
Parts:
- PIR1, PIR2: footprint Connector_PinHeader_2.54mm:PinHeader_1x03_P2.54mm_Vertical -> Connector_JST:JST_EH_B3B-EH-A_1x03_P2.50mm_Vertical
Changed lines of the file:
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@@
       (effects (font (size 1.27 1.27)))
     )
-    (property "Footprint" "Connector_PinHeader_2.54mm:PinHeader_1x03_P2.54mm_Vertical" (at 156.083 45.212 0)
+    (property "Footprint" "Connector_JST:JST_EH_B3B-EH-A_1x03_P2.50mm_Vertical" (at 156.083 45.212 0)
       (effects (font (size 1.27 1.27)) hide)
     )
@@
       (effects (font (size 1.27 1.27)))
     )
-    (property "Footprint" "Connector_PinHeader_2.54mm:PinHeader_1x03_P2.54mm_Vertical" (at 102.87 45.72 0)
+    (property "Footprint" "Connector_JST:JST_EH_B3B-EH-A_1x03_P2.50mm_Vertical" (at 102.87 45.72 0)
       (effects (font (size 1.27 1.27)) hide)
     )
