File: PCB-light-challenge/LEDS.kicad_sch (KiCad schematic)
At the start: 0 parts

Commit message: Footprints toegevoegd van alles
Other:
- company: (none) -> HHS Living Labs
Changed lines of the file:
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@@
 (kicad_sch (version 20230121) (generator eeschema)
   (paper "A4")
+  (title_block
+    (date "2023-11-06")
+    (rev "V0.1")
+    (company "HHS Living Labs")
+  )
 )
