File: PCB-light-challenge/_autosave-PCB-light-challenge.kicad_pcb (KiCad board)
At the start: 4 copper layers, 80.1 x 79.1 mm, 24 parts, among them J1 Conn_01x16_Socket, J2 Conn_01x16_Socket, U2 AP9101CK, U3 SP8K32FRATB

Commit message: EDS protection en fuse toegevoegd
we moeten nog wel footprints checken
Parts:
- added 230VAC1: Screw_Terminal_01x02, TerminalBlock_4Ucon:TerminalBlock_4Ucon_1x02_P3.50mm_Vertical, F.Cu at (241.6, 91.6)
Changed lines of the file:
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@@
       (net 45 "Net-(230VAC1-Pin_1)") (pinfunction "AC_IN_(N)") (pintype "input") (solder_mask_margin 0.102))
+  )
+  (footprint "TerminalBlock_4Ucon:TerminalBlock_4Ucon_1x02_P3.50mm_Vertical" (layer "F.Cu")
+    (at 241.61 91.625)
+    (descr "Terminal Block 4Ucon ItemNo. 10693, vertical (cable from top), 2 pins, pitch 3.5mm, size 8x8.3mm^2, drill diamater 1.3mm, pad diameter 2.6mm, see http://www.4uconnector.com/online/object/4udrawing/10693.pdf, script-generated with , script-generated using https://github.com/pointhi/kicad-footprint-generator/scripts/TerminalBlock_4Ucon")
+    (tags "THT Terminal Block 4Ucon ItemNo. 10693 vertical pitch 3.5mm size 8x8.3mm^2 drill 1.3mm pad 2.6mm")
+    (property "Sheetfile" "Battery_charger.kicad_sch")
+    (property "Sheetname" "Battery_charger")
+    (property "ki_description" "Generic screw terminal, single row, 01x02, script generated (kicad-library-utils/schlib/autogen/connector/)")
+    (property "ki_keywords" "screw terminal")
+    (attr through_hole)
+    (fp_text reference "230VAC1" (at 1.75 -4.76) (layer "F.SilkS")
+        (effects (font (size 1 1) (thickness 0.15)))
+    )
+    (fp_text value "Screw_Terminal_01x02" (at 1.75 5.66) (layer "F.Fab")
+        (effects (font (size 1 1) (thickness 0.15)))
+    )
+    (fp_text user "${REFERENCE}" (at 1.75 3.45) (layer "F.Fab")
+        (effects (font (size 1 1) (thickness 0.15)))
+    )
+    (fp_line (start -2.55 2.66) (end -2.55 4.9)
+      (stroke (width 0.12) (type solid)) (layer "F.SilkS"))
+    (fp_line (start -2.55 4.9) (end -0.55 4.9)
+      (stroke (width 0.12) (type solid)) (layer "F.SilkS"))
+    (fp_line (start -2.31 -3.76) (end -2.31 4.66)
+      (stroke (width 0.12) (type solid)) (layer "F.SilkS"))
+    (fp_line (start -2.31 -3.76) (end 5.81 -3.76)
+      (stroke (width 0.12) (type solid)) (layer "F.SilkS"))
+    (fp_line (start -2.31 1.101) (end -1.54 1.101)
+      (stroke (width 0.12) (type solid)) (layer "F.SilkS"))
+    (fp_line (start -2.31 4.66) (end 5.81 4.66)
+      (stroke (width 0.12) (type solid)) (layer "F.SilkS"))
+    (fp_line (start -1.4 -3) (end -1.4 -1.54)
+      (stroke (width 0.12) (type solid)) (layer "F.SilkS"))
+    (fp_line (start -1.4 -3) (end 1.4 -3)
+      (stroke (width 0.12) (type solid)) (layer "F.SilkS"))
+    (fp_line (start 1.4 -3) (end 1.4 -1.54)
+      (stroke (width 0.12) (type solid)) (layer "F.SilkS"))
+    (fp_line (start 1.54 1.101) (end 2.367 1.101)
+      (stroke (width 0.12) (type solid)) (layer "F.SilkS"))
+    (fp_line (start 2.1 -3) (end 2.1 -0.689)
+      (stroke (width 0.12) (type solid)) (layer "F.SilkS"))
+    (fp_line (start 2.1 -3) (end 4.9 -3)
+      (stroke (width 0.12) (type solid)) (layer "F.SilkS"))
+    (fp_line (start 2.1 0.689) (end 2.1 0.75)
+      (stroke (width 0.12) (type solid)) (layer "F.SilkS"))
+    (fp_line (start 2.1 0.75) (end 2.101 0.75)
+      (stroke (width 0.12) (type solid)) (layer "F.SilkS"))
+    (fp_line (start 4.634 1.101) (end 5.81 1.101)
+      (stroke (width 0.12) (type solid)) (layer "F.SilkS"))
+    (fp_line (start 4.9 -3) (end 4.9 -0.689)
+      (stroke (width 0.12) (type solid)) (layer "F.SilkS"))
+    (fp_line (start 4.9 0.689) (end 4.9 0.75)
+      (stroke (width 0.12) (type solid)) (layer "F.SilkS"))
+    (fp_line (start 4.9 0.75) (end 4.9 0.75)
+      (stroke (width 0.12) (type solid)) (layer "F.SilkS"))
+    (fp_line (start 5.81 -3.76) (end 5.81 4.66)
+      (stroke (width 0.12) (type solid)) (layer "F.SilkS"))
+    (fp_arc (start -0.99789 -1.529434) (mid -0.000785 -2.600382) (end 0.998 -1.531)
+      (stroke (width 0.12) (type solid)) (layer "F.SilkS"))
+    (fp_arc (start 2.560085 -1.257767) (mid 3.499876 -2.600282) (end 4.44 -1.258)
+      (stroke (width 0.12) (type solid)) (layer "F.SilkS"))
+    (fp_line (start -2.75 -4.2) (end -2.75 5.11)
+      (stroke (width 0.05) (type solid)) (layer "F.CrtYd"))
+    (fp_line (start -2.75 5.11) (end 6.25 5.11)
+      (stroke (width 0.05) (type solid)) (layer "F.CrtYd"))
+    (fp_line (start 6.25 -4.2) (end -2.75 -4.2)
+      (stroke (width 0.05) (type solid)) (layer "F.CrtYd"))
+    (fp_line (start 6.25 5.11) (end 6.25 -4.2)
+      (stroke (width 0.05) (type solid)) (layer "F.CrtYd"))
+    (fp_line (start -2.25 -3.7) (end 5.75 -3.7)
+      (stroke (width 0.1) (type solid)) (layer "F.Fab"))
+    (fp_line (start -2.25 1.1) (end 5.75 1.1)
+      (stroke (width 0.1) (type solid)) (layer "F.Fab"))
+    (fp_line (start -2.25 2.6) (end -2.25 -3.7)
+      (stroke (width 0.1) (type solid)) (layer "F.Fab"))
+    (fp_line (start -1.4 -3) (end -1.4 0.75)
+      (stroke (width 0.1) (type solid)) (layer "F.Fab"))
+    (fp_line (start -1.4 0.75) (end 1.4 0.75)
+      (stroke (width 0.1) (type solid)) (layer "F.Fab"))
+    (fp_line (start -0.25 4.6) (end -2.25 2.6)
+      (stroke (width 0.1) (type solid)) (layer "F.Fab"))
+    (fp_line (start 1.4 -3) (end -1.4 -3)
+      (stroke (width 0.1) (type solid)) (layer "F.Fab"))
+    (fp_line (start 1.4 0.75) (end 1.4 -3)
+      (stroke (width 0.1) (type solid)) (layer "F.Fab"))
+    (fp_line (start 2.1 -3) (end 2.1 0.75)
+      (stroke (width 0.1) (type solid)) (layer "F.Fab"))
+    (fp_line (start 2.1 0.75) (end 4.9 0.75)
+      (stroke (width 0.1) (type solid)) (layer "F.Fab"))
+    (fp_line (start 4.9 -3) (end 2.1 -3)
+      (stroke (width 0.1) (type solid)) (layer "F.Fab"))
+    (fp_line (start 4.9 0.75) (end 4.9 -3)
+      (stroke (width 0.1) (type solid)) (layer "F.Fab"))
+    (fp_line (start 5.75 -3.7) (end 5.75 4.6)
+      (stroke (width 0.1) (type solid)) (layer "F.Fab"))
+    (fp_line (start 5.75 4.6) (end -0.25 4.6)
+      (stroke (width 0.1) (type solid)) (layer "F.Fab"))
+    (fp_circle (center 0 -1.6) (end 1 -1.6)
+      (stroke (width 0.1) (type solid)) (fill none) (layer "F.Fab"))
+    (fp_circle (center 3.5 -1.6) (end 4.5 -1.6)
+      (stroke (width 0.1) (type solid)) (fill none) (layer "F.Fab"))
+    (pad "1" thru_hole rect (at 0 0) (size 2.6 2.6) (drill 1.3) (layers "*.Cu" "*.Mask")
+      (net 45 "Net-(230VAC1-Pin_1)") (pinfunction "Pin_1") (pintype "passive"))
+    (pad "2" thru_hole circle (at 3.5 0) (size 2.6 2.6) (drill 1.3) (layers "*.Cu" "*.Mask")
+      (net 44 "Net-(230VAC1-Pin_2)") (pinfunction "Pin_2") (pintype "passive"))
+    (model "${KICAD6_3DMODEL_DIR}/TerminalBlock_4Ucon.3dshapes/TerminalBlock_4Ucon_1x02_P3.50mm_Vertical.wrl"
+      (offset (xyz 0 0 0))
+      (scale (xyz 1 1 1))
+      (rotate (xyz 0 0 0))
+    )
   )
   (footprint "Diode_SMD:D_SOD-323_HandSoldering" (layer "F.Cu")
