File: PCB-light-challenge/Micro_Controller.kicad_sch (KiCad schematic)
At the start: 11 parts, among them J1 Conn_01x16_Socket, J2 Conn_01x16_Socket

Commit message: PCB 80% af
Parts:
- removed J2: Conn_01x16_Socket, Connector_PinHeader_2.54mm:PinHeader_1x16_P2.54mm_Vertical, symbol Connector:Conn_01x16_Socket
- added J3: Conn_01x13_Socket, Connector_PinHeader_2.54mm:PinHeader_1x13_P2.54mm_Vertical, symbol Connector:Conn_01x13_Socket
- Batterij1: footprint Connector_PinHeader_2.54mm:PinHeader_1x02_P2.54mm_Horizontal -> TerminalBlock_TE-Connectivity:TerminalBlock_TE_282834-2_1x02_P2.54mm_Horizontal
Connections:
- net GND: no longer U-PICO1. (SWDIO)
- net GP10: now also J3.6 (Pin_6)
- net GP11: now also J3.5 (Pin_5)
- net GP12: now also J3.4 (Pin_4)
- net GP13: now also J3.3 (Pin_3)
- net GP14: now also J3.2 (Pin_2)
- net GP15: now also J3.1 (Pin_1)
- net GP16: now also J1.6 (Pin_6); no longer J1.1 (Pin_1)
- net GP17: now also J1.5 (Pin_5); no longer J1.2 (Pin_2)
- net GP18: now also J1.4 (Pin_4); no longer J1.3 (Pin_3)
- net GP19: now also J1.3 (Pin_3); no longer J1.4 (Pin_4)
- net GP20: now also J1.2 (Pin_2); no longer J1.5 (Pin_5)
- net GP21: now also J1.1 (Pin_1); no longer J1.6 (Pin_6)
- net GP3: now also J3.13 (Pin_13)
- net GP4: now also J3.12 (Pin_12)
- net GP5: now also J3.11 (Pin_11)
- net GP6: now also J3.10 (Pin_10)
- net GP7: now also J3.9 (Pin_9)
- net GP8: now also J3.8 (Pin_8)
- net GP9: now also J3.7 (Pin_7)
- no-connect marks 2 -> 0
